Commit message: 让机械臂离地0.55米，管道距离机械臂1米

File: robots/z1_description/xacro/robot.xacro (robot description, xacro)
@@ -8,5 +8,5 @@
     <link name="world"/>
     <joint name="base_static_joint" type="fixed">
-        <origin rpy="0 0 0" xyz="0 0 0"/>
+        <origin rpy="0 0 0" xyz="0 0 0.55"/>
         <parent link="world"/>
         <child link="link00"/>
@@ -25,5 +25,5 @@
     </link>
     <joint name="world_to_combine_joint" type="fixed">
-        <origin xyz="1 0 0.2" rpy="0 0 1.5708"/>
+        <origin xyz="1.0 0 0.025" rpy="0 0 1.5708"/>
         <parent link="link00"/>
         <child link="combine_link"/>

Commit message: 10.11修复bug

File: robots/z1_description/xacro/robot.xacro (robot description, xacro)
@@ -8,5 +8,5 @@
     <link name="world"/>
     <joint name="base_static_joint" type="fixed">
-        <origin rpy="0 0 0" xyz="0 0 0.55"/>
+        <origin rpy="0 0 0" xyz="0 0 0.6"/>
         <parent link="world"/>
         <child link="link00"/>
@@ -25,5 +25,5 @@
     </link>
     <joint name="world_to_combine_joint" type="fixed">
-        <origin xyz="1.0 0 0.025" rpy="0 0 1.5708"/>
+        <origin xyz="1.0 0 0.075" rpy="0 0 1.5708"/>
         <parent link="link00"/>
         <child link="combine_link"/>
