Commit message: 10.8 加入管道模型,修改相机安装位置

File: robots/z1_description/xacro/camera.xacro (robot description, xacro)
@@ -4,5 +4,5 @@
     <link name="camera_link">
       <visual>
-        <origin xyz="0.05 0 0" rpy="0 0 1.5708"/>
+        <origin xyz="0 0 0" rpy="0 0 1.5708"/>
         <geometry>
           <mesh filename="package://realsense2_description/meshes/d435.dae" />
@@ -13,5 +13,6 @@
         <origin xyz="0 0 0" rpy="0 0 0"/>
         <geometry>
-          <box size="0.02 0.05 0.05"/>
+          <!-- <box size="0.02 0.05 0.05"/> -->
+          <box size="0.0 0.0 0.0"/>
         </geometry>
       </collision>
@@ -24,5 +25,5 @@
       <parent link="${parent}"/>
       <child link="camera_link"/>
-      <origin xyz="0.05 0 0.05" rpy="0 0 0"/>
+      <origin xyz="0.0389 0 -0.0389" rpy="0 0.7854 0"/>
     </joint>
     <link name="camera_optical_frame"/>
@@ -32,36 +33,4 @@
       <origin xyz="0 0 0" rpy="-1.5708 0 -1.5708"/>
     </joint>
-    <!-- <gazebo reference="camera_link">
-      <material>Gazebo/Black</material>
-      <sensor type="camera" name="gripper_camera_sensor">
-        <update_rate>30.0</update_rate>
-        <camera name="head">
-          <horizontal_fov>1.3962634</horizontal_fov>
-          <image>
-            <width>800</width>
-            <height>800</height>
-            <format>R8G8B8</format>
-          </image>
-          <clip>
-            <near>0.02</near>
-            <far>300</far>
-          </clip>
-        </camera>
-        <plugin name="camera_controller" filename="libgazebo_ros_camera.so">
-          <alwaysOn>true</alwaysOn>
-          <updateRate>0.0</updateRate>
-          <cameraName>z1/camera</cameraName>
-          <imageTopicName>image_raw</imageTopicName>
-          <cameraInfoTopicName>camera_info</cameraInfoTopicName>
-          <frameName>camera_optical_frame</frameName>
-          <hackBaseline>0.07</hackBaseline>
-          <distortionK1>0.0</distortionK1>
-          <distortionK2>0.0</distortionK2>
-          <distortionK3>0.0</distortionK3>
-          <distortionT1>0.0</distortionT1>
-          <distortionT2>0.0</distortionT2>
-        </plugin>
-      </sensor>
-    </gazebo> -->
     <gazebo reference="camera_link">
       <material>Gazebo/Black</material>
@@ -95,4 +64,11 @@
         </plugin>
       </sensor>
+      <collision>
+        <surface>
+          <contact>
+            <collide_bitmask>0x01</collide_bitmask>
+          </contact>
+        </surface>
+      </collision>
     </gazebo>
   </xacro:macro>

File: robots/z1_description/xacro/robot.xacro (robot description, xacro)
@@ -11,4 +11,21 @@
         <parent link="world"/>
         <child link="link00"/>
+    </joint>
+    <link name="combine_link">
+        <visual name="visual">
+            <geometry>
+                <mesh filename="package://z1_description/meshes/visual/combine.dae" scale="1 1 1"/>
+            </geometry>
+        </visual>
+        <collision name="collision">
+            <geometry>
+                <mesh filename="package://z1_description/meshes/collision/combine.stl" scale="1 1 1"/>
+            </geometry>
+        </collision>
+    </link>
+    <joint name="world_to_combine_joint" type="fixed">
+        <origin xyz="1 0 0.2" rpy="0 0 1.5708"/>
+        <parent link="link00"/>
+        <child link="combine_link"/>
     </joint>
     <link name="link00">
@@ -280,4 +297,11 @@
         <gazebo reference="gripperMover">
             <self_collide>true</self_collide>
+            <collision>
+                <surface>
+                <contact>
+                    <collide_bitmask>0x01</collide_bitmask>
+                </contact>
+                </surface>
+            </collision>
         </gazebo>
     </xacro:if>

Commit message: add d435.dae model

File: robots/z1_description/xacro/camera.xacro (robot description, xacro)
@@ -6,5 +6,5 @@
         <origin xyz="0 0 0" rpy="0 0 1.5708"/>
         <geometry>
-          <mesh filename="package://realsense2_description/meshes/d435.dae" />
+          <mesh filename="package://z1_description/meshes/visual/d435.dae" />
         </geometry>
         <!-- <material name="black"/> -->
