Commit message: update combine env

File: robots/z1_description/urdf/z1.urdf (robot description, URDF)
Before this commit: robot z1_description, 8 links, 7 joints
Links:
- added link camera_link, mass 0.01; collision box size=0.0 0.0 0.0; visual mesh filename=package://z1_description/meshes/visual//d435.dae
- added link camera_optical_frame
- added link gripperMover, mass 0.27621302
- added link gripperStator, mass 0.52603655
Joints:
- added joint camera_joint: type fixed, parent gripperMover, child camera_link, origin xyz=0.0389 0 -0.0389 rpy=0 0.7854 0
- added joint camera_optical_joint: type fixed, parent camera_link, child camera_optical_frame, origin xyz=0 0 0 rpy=-1.5708 0 -1.5708
- added joint gripperStator: type fixed, parent link06, child gripperStator, origin xyz=0.051 0.0 0.0 rpy=0 0 0
- added joint jointGripper: type revolute, parent gripperStator, child gripperMover, origin xyz=0.049 0.0 0 rpy=0 0 0, axis 0 1 0, limit lower=-1.5707963267948966 upper=0.0 effort=30.0 velocity=3.1415

File: robots/z1_description/xacro/robot_combine.xacro (robot description, xacro)
@@ -12,21 +12,21 @@
         <child link="link00"/>
     </joint>
-    <!-- <link name="flower_link">
+    <link name="combine_link">
         <visual name="visual">
             <geometry>
-                <mesh filename="package://z1_description/meshes/visual/flower.dae" scale="1 1 1"/>
+                <mesh filename="package://z1_description/meshes/visual/combine.dae" scale="1 1 1"/>
             </geometry>
         </visual>
         <collision name="collision">
             <geometry>
-                <mesh filename="package://z1_description/meshes/collision/flower.stl" scale="1 1 1"/>
-            </geometry>
-        </collision>
-    </link>
-    <joint name="link00_to_flower_joint" type="fixed">
-        <origin xyz="0.75 0.0 0.2" rpy="0.2 -1.56 0.0"/>
+                <mesh filename="package://z1_description/meshes/collision/combine.stl" scale="1 1 1"/>
+            </geometry>
+        </collision>
+    </link>
+    <joint name="world_to_combine_joint" type="fixed">
+        <origin xyz="0.85 0.0 0.0" rpy="0.7 0.1 1.5708"/>
         <parent link="link00"/>
-        <child link="flower_link"/>
-    </joint> -->
+        <child link="combine_link"/>
+    </joint>
     <link name="link00">
         <visual>
@@ -312,6 +312,4 @@
     <xacro:motorTransmission name="5"/>
     <xacro:motorTransmission name="6"/>
-<xacro:if value="$(arg UnitreeGripper)">
-    <xacro:gripper_camera parent="gripperMover" />
-</xacro:if>
+<xacro:gripper_camera parent="gripperMover" />
 </robot>

File: robots/z1_description/xacro/robot_flower.xacro (robot description, xacro)
@@ -12,5 +12,5 @@
         <child link="link00"/>
     </joint>
-    <!-- <link name="flower_link">
+    <link name="flower_link">
         <visual name="visual">
             <geometry>
@@ -25,8 +25,8 @@
     </link>
     <joint name="link00_to_flower_joint" type="fixed">
-        <origin xyz="0.75 0.0 0.2" rpy="0.2 -1.56 0.0"/>
+        <origin xyz="0.8 0.0 0.2" rpy="0.0 -1.46 0.0"/>
         <parent link="link00"/>
         <child link="flower_link"/>
-    </joint> -->
+    </joint>
     <link name="link00">
         <visual>
@@ -312,6 +312,4 @@
     <xacro:motorTransmission name="5"/>
     <xacro:motorTransmission name="6"/>
-<xacro:if value="$(arg UnitreeGripper)">
-    <xacro:gripper_camera parent="gripperMover" />
-</xacro:if>
+<xacro:gripper_camera parent="gripperMover" />
 </robot>
